Commit message: Fix rosbot3 xacro file

File: urdf/rosbot3.xacro (robot description, xacro)
@@ -42,5 +42,5 @@
     parent="base_link"
     child="chassis"
-    z="${ground_clearance + 0.5 * body_height}"
+    z="${ground_clearance + 0.5 * chassis_height}"
   />
   <xacro:solid_block
@@ -50,15 +50,16 @@
     size_z="${chassis_height}"
   />
+  <link name="payload_base"/>
   <xacro:joint_fixed
     parent="chassis"
     child="payload_base"
-    z="${0.5 * body_height}"
+    z="${0.5 * chassis_height}"
   />
-  <xacro:solid_block
+  <!-- <xacro:solid_block
     name="camera_support"
     size_x="${camera_width}"
     size_y="${camera_depth}"
     size_z="${camera_height}"
-  />
+  /> -->
   <xacro:camera_link name="camera_front"/>
   <xacro:joint_fixed

Commit message: Add wheels to robot model

File: urdf/rosbot3.xacro (robot description, xacro)
@@ -2,5 +2,5 @@
 <!--
   Description of the ROSbot3 robot.
-  Author: Helio Perroni Filho
+  Author: Breno Uliana de Angelo
 -->
 <robot name="rosbot3" xmlns:xacro="http://www.ros.org/wiki/xacro">
@@ -21,4 +21,5 @@
   <!-- Picking a random but reasonable value -->
   <xacro:property name="wheel_width" value="${30.0 * M}"/> <!-- Not provided in the manual -->
+  <xacro:property name="wheel_axle_z_offset" value="${wheel_diameter * 0.5 - 0.5 * chassis_height - ground_clearance}"/>
   <!-- Dimensions of the robot main body -->
   <xacro:property name="chassis_length" value="${200.0 * M}"/>
@@ -38,4 +39,5 @@
   <xacro:property name="lidar_displacement_x" value="${0.0 * M}"/> <!-- Not provided in the manual -->
   <xacro:property name="lidar_displacement_z" value="${overall_height_with_lidar - overall_height - lidar_height * 0.5 }"/>
+  <!-- Chassis -->
   <link name="base_link"/>
   <xacro:joint_fixed
@@ -56,4 +58,57 @@
     z="${0.5 * chassis_height}"
   />
+  <!-- Wheels -->
+  <xacro:macro
+    name="wheels"
+    params="position"
+  >
+    <xacro:solid_cylinder
+      name="wheel_${position}_left"
+      length="${wheel_width}"
+      radius="${wheel_diameter * 0.5}"
+      roll="${90.0 * DEG}"
+    />
+    <xacro:solid_cylinder
+      name="wheel_${position}_right"
+      length="${wheel_width}"
+      radius="${wheel_diameter * 0.5}"
+      roll="${90.0 * DEG}"
+    />
+    <xacro:solid_cylinder
+      name="wheel_${position}_axle"
+      length="${chassis_width}"
+      radius="0.005"
+      roll="${90.0 * DEG}"
+    />
+    <xacro:joint_continuous
+      name="joint_wheel_${position}_left"
+      parent="wheel_${position}_axle"
+      child="wheel_${position}_left"
+      y="${(chassis_width + wheel_width) * 0.5}"
+      axis="0 1 0"
+    />
+    <xacro:joint_continuous
+      name="joint_wheel_${position}_right"
+      parent="wheel_${position}_axle"
+      child="wheel_${position}_right"
+      y="${(chassis_width + wheel_width) * -0.5}"
+      axis="0 1 0"
+    />
+  </xacro:macro>
+  <xacro:wheels position="front"/>
+  <xacro:wheels position="rear"/>
+  <xacro:joint_fixed
+    parent="chassis"
+    child="wheel_front_axle"
+    x="${0.5 * wheel_wheelbase}"
+    z="${wheel_axle_z_offset}"
+  />
+  <xacro:joint_fixed
+    parent="chassis"
+    child="wheel_rear_axle"
+    x="${-0.5 * wheel_wheelbase}"
+    z="${wheel_axle_z_offset}"
+  />
+  <!-- Camera -->
   <!-- <xacro:solid_block
     name="camera_support"
@@ -69,4 +124,5 @@
     z="${camera_displacement_z}"
   />
+  <!-- LiDAR -->
   <xacro:solid_cylinder
     name="lidar"

Commit message: Split robot description into base and sensors

File: urdf/rosbot3.xacro (robot description, xacro)
@@ -1,5 +1,5 @@
 <?xml version="1.0" encoding="utf-8"?>
 <!--
-  Description of the ROSbot3 robot.
+  Complete description of the ROSbot3 robot.
   Author: Breno Uliana de Angelo
 -->
@@ -7,138 +7,5 @@
   <xacro:include filename="$(find ros_commons)/urdf/domain.xacro"/>
   <xacro:property name="M" value="0.001"/>
-  <!-- Overall height of the robot body without camera and LiDAR -->
-  <xacro:property name="overall_height" value="${103.0 * M}"/>
-  <!-- Total height including the camera support -->
-  <xacro:property name="overall_height_with_camera_support" value="${197.0 * M}"/>
-  <!-- Total height including the LiDAR -->
-  <xacro:property name="overall_height_with_lidar" value="${141.0 * M}"/>
-  <!-- Height the chassis is above the ground -->
-  <xacro:property name="ground_clearance" value="${23.0 * M}"/>
-  <!-- Using standard wheels -->
-  <xacro:property name="wheel_diameter" value="${84.0 * M}"/>
-  <xacro:property name="wheel_wheelbase" value="${106.0 * M}"/>
-  <!-- Wheel width is not provided in the manual https://husarion.com/manuals/rosbot -->
-  <!-- Picking a random but reasonable value -->
-  <xacro:property name="wheel_width" value="${30.0 * M}"/> <!-- Not provided in the manual -->
-  <xacro:property name="wheel_axle_z_offset" value="${wheel_diameter * 0.5 - 0.5 * chassis_height - ground_clearance}"/>
-  <!-- Dimensions of the robot main body -->
-  <xacro:property name="chassis_length" value="${200.0 * M}"/>
-  <xacro:property name="chassis_width" value="${233.0 * M}"/>
-  <xacro:property name="chassis_height" value="${overall_height - ground_clearance}"/>
-  <!-- Dimensions of the camera itself -->
-  <xacro:property name="camera_height" value="${30.0 * M}"/> <!-- Not provided in the manual -->
-  <xacro:property name="camera_width" value="${80.0 * M}"/> <!-- Not provided in the manual -->
-  <xacro:property name="camera_depth" value="${15.0 * M}"/> <!-- Not provided in the manual -->
-  <!-- Camera position relative to the payload base -->
-  <xacro:property name="camera_displacement_x" value="${0.0 * M}"/> <!-- Not provided in the manual -->
-  <xacro:property name="camera_displacement_z" value="${overall_height_with_camera_support - overall_height - camera_height * 0.5 }"/>
-  <!-- Dimensions of the LiDAR itself -->
-  <xacro:property name="lidar_diameter" value="${80.0 * M}"/>
-  <xacro:property name="lidar_height" value="${overall_height_with_lidar - overall_height_with_camera_support}"/>
-  <!-- LiDAR position relative to the payload base -->
-  <xacro:property name="lidar_displacement_x" value="${0.0 * M}"/> <!-- Not provided in the manual -->
-  <xacro:property name="lidar_displacement_z" value="${overall_height_with_lidar - overall_height - lidar_height * 0.5 }"/>
-  <!-- Chassis -->
-  <link name="base_link"/>
-  <xacro:joint_fixed
-    parent="base_link"
-    child="chassis"
-    z="${ground_clearance + 0.5 * chassis_height}"
-  />
-  <xacro:solid_block
-    name="chassis"
-    size_x="${chassis_length}"
-    size_y="${chassis_width}"
-    size_z="${chassis_height}"
-  />
-  <link name="payload_base"/>
-  <xacro:joint_fixed
-    parent="chassis"
-    child="payload_base"
-    z="${0.5 * chassis_height}"
-  />
-  <!-- Wheels -->
-  <xacro:macro
-    name="wheels"
-    params="position"
-  >
-    <xacro:solid_cylinder
-      name="wheel_${position}_left"
-      length="${wheel_width}"
-      radius="${wheel_diameter * 0.5}"
-      roll="${90.0 * DEG}"
-    />
-    <xacro:solid_cylinder
-      name="wheel_${position}_right"
-      length="${wheel_width}"
-      radius="${wheel_diameter * 0.5}"
-      roll="${90.0 * DEG}"
-    />
-    <xacro:solid_cylinder
-      name="wheel_${position}_axle"
-      length="${chassis_width}"
-      radius="0.005"
-      roll="${90.0 * DEG}"
-    />
-    <xacro:joint_continuous
-      name="joint_wheel_${position}_left"
-      parent="wheel_${position}_axle"
-      child="wheel_${position}_left"
-      y="${(chassis_width + wheel_width) * 0.5}"
-      axis="0 1 0"
-    />
-    <xacro:joint_continuous
-      name="joint_wheel_${position}_right"
-      parent="wheel_${position}_axle"
-      child="wheel_${position}_right"
-      y="${(chassis_width + wheel_width) * -0.5}"
-      axis="0 1 0"
-    />
-  </xacro:macro>
-  <xacro:wheels position="front"/>
-  <xacro:wheels position="rear"/>
-  <xacro:joint_fixed
-    parent="chassis"
-    child="wheel_front_axle"
-    x="${0.5 * wheel_wheelbase}"
-    z="${wheel_axle_z_offset}"
-  />
-  <xacro:joint_fixed
-    parent="chassis"
-    child="wheel_rear_axle"
-    x="${-0.5 * wheel_wheelbase}"
-    z="${wheel_axle_z_offset}"
-  />
-  <!-- Camera -->
-  <!-- <xacro:solid_block
-    name="camera_support"
-    size_x="${camera_width}"
-    size_y="${camera_depth}"
-    size_z="${camera_height}"
-  /> -->
-  <xacro:camera_link name="camera_front"/>
-  <xacro:joint_fixed
-    parent="payload_base"
-    child="camera_front"
-    x="${camera_displacement_x}"
-    z="${camera_displacement_z}"
-  />
-  <!-- LiDAR -->
-  <xacro:solid_cylinder
-    name="lidar"
-    radius="${lidar_diameter * 0.5}"
-    length="${lidar_height}"
-  />
-  <xacro:joint_fixed
-    parent="payload_base"
-    child="lidar"
-    x="${lidar_displacement_x}"
-    z="${lidar_displacement_z}"
-  />
-  <link name="laser"/>
-  <xacro:joint_fixed
-    parent="lidar"
-    child="laser"
-    z="${0.5 * lidar_height}"
-  />
+  <xacro:include filename="$(find rosbot3_description)/urdf/base.xacro"/>
+  <xacro:include filename="$(find rosbot3_description)/urdf/sensors.xacro"/>
 </robot>
