Commit message: Include camera support in robot description

File: urdf/sensors.xacro (robot description, xacro)
@@ -9,30 +9,61 @@
   <!-- Total height including the LiDAR -->
   <xacro:property name="overall_height_with_lidar" value="${141.0 * M}"/>
-  <!-- Dimensions of the camera itself -->
-  <xacro:property name="camera_height" value="${30.0 * M}"/> <!-- Not provided in the manual -->
-  <xacro:property name="camera_width" value="${80.0 * M}"/> <!-- Not provided in the manual -->
-  <xacro:property name="camera_depth" value="${15.0 * M}"/> <!-- Not provided in the manual -->
+  <!-- Dimensions of the camera itself, retrieved from https://shop.luxonis.com/products/oak-d?srsltid=AfmBOor06MUSThj6dwPJDxshBfcSD2IxSXlwf0L-gUbfsm9e8RdP_7_F -->
+  <xacro:property name="camera_height" value="${54.5 * M}"/>
+  <xacro:property name="camera_width" value="${110.0 * M}"/>
+  <xacro:property name="camera_depth" value="${33.0 * M}"/>
   <!-- Camera position relative to the payload base -->
   <xacro:property name="camera_displacement_x" value="${0.0 * M}"/> <!-- Not provided in the manual -->
   <xacro:property name="camera_displacement_z" value="${overall_height_with_camera_support - overall_height - camera_height * 0.5 }"/>
-  <!-- Dimensions of the LiDAR itself -->
-  <xacro:property name="lidar_diameter" value="${80.0 * M}"/>
-  <xacro:property name="lidar_height" value="${overall_height_with_lidar - overall_height_with_camera_support}"/>
+  <!-- Camera support -->
+  <xacro:property name="camera_support_edge" value="${10.0 * M}"/>
+  <xacro:property name="camera_support_displacement_from_camera" value="${40.0 * M}"/>
+  <xacro:property name="camera_support_height" value="${camera_displacement_z + camera_support_edge * 0.5}"/>
+  <!-- Dimensions of the LiDAR itself
+       According to https://www.slamtec.com/en/C1/Spec the LiDAR is 55.6 x 55.6 x 41.3mm with rectangular base.
+       Approximating to a cylinder with diameter 55.6mm.
+       The height of the LiDAR is the total height of the robot body without the camera support.
+  -->
+  <xacro:property name="lidar_diameter" value="${55.6 * M}"/>
+  <xacro:property name="lidar_height" value="${overall_height_with_lidar - overall_height}"/>
   <!-- LiDAR position relative to the payload base -->
   <xacro:property name="lidar_displacement_x" value="${0.0 * M}"/> <!-- Not provided in the manual -->
   <xacro:property name="lidar_displacement_z" value="${overall_height_with_lidar - overall_height - lidar_height * 0.5 }"/>
   <!-- Camera -->
-  <!-- <xacro:solid_block
-    name="camera_support"
-    size_x="${camera_width}"
-    size_y="${camera_depth}"
+  <xacro:solid_block
+    name="camera_front"
+    size_x="${camera_depth}"
+    size_y="${camera_width}"
     size_z="${camera_height}"
-  /> -->
+  />
   <xacro:camera_link name="camera_front"/>
+  <xacro:solid_block
+    name="camera_support_vertical"
+    size_x="${camera_support_edge}"
+    size_y="${camera_support_edge}"
+    size_z="${camera_support_height}"
+  />
+  <xacro:solid_block
+    name="camera_support_horizontal"
+    size_x="${camera_support_displacement_from_camera}"
+    size_y="${camera_support_edge}"
+    size_z="${camera_support_edge}"
+  />
   <xacro:joint_fixed
     parent="payload_base"
+    child="camera_support_vertical"
+    x="${-(camera_displacement_x + camera_depth + camera_support_edge * 0.5 + camera_support_displacement_from_camera)}"
+    z="${camera_support_height * 0.5}"
+  />
+  <xacro:joint_fixed
+    parent="camera_support_vertical"
+    child="camera_support_horizontal"
+    x="${(camera_support_displacement_from_camera - camera_support_edge) * 0.5}"
+    z="${(camera_support_height + camera_support_edge) * 0.5}"
+  />
+  <xacro:joint_fixed
+    parent="camera_support_horizontal"
     child="camera_front"
-    x="${camera_displacement_x}"
-    z="${camera_displacement_z}"
+    x="${camera_support_displacement_from_camera * 0.5 + camera_depth * 0.5}"
   />
   <!-- LiDAR -->
